File: attiny85 programmer/attiny85 programmer.kicad_pcb (KiCad board)
At the start: 2 copper layers, 69.8 x 45.7 mm, 13 parts

Commit message: adjust position of bootloader burning socket
Parts:
- moved REF** 7.62 mm to (121.9, 86.4)
Changed lines of the file:
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@@
 	(footprint "Package_DIP:DIP-8_W7.62mm"
 		(layer "F.Cu")
-		(at 121.92 93.98)
+		(at 121.92 86.36)
 		(descr "8-lead though-hole mounted DIP package, row spacing 7.62 mm (300 mils)")
 		(tags "THT DIP DIL PDIP 2.54mm 7.62mm 300mil")
@@
 	)
 	(gr_text "Burn\nBootloader"
-		(at 125.73 91.44 0)
+		(at 125.73 100.33 0)
 		(layer "F.SilkS")
 		(effects
@@
 	)
 	(segment
+		(start 119.38 96.52)
+		(end 121.92 93.98)
+		(width 1)
+		(layer "F.Cu")
+		(net 0)
+	)
+	(segment
 		(start 177.8 101.6)
 		(end 177.8 97.79)
@@
 	)
 	(segment
-		(start 119.38 104.14)
-		(end 121.92 101.6)
-		(width 1)
-		(layer "F.Cu")
-		(net 0)
-	)
-	(segment
-		(start 134.62 83.82)
-		(end 137.16 83.82)
+		(start 160.02 88.9)
+		(end 160.02 93.98)
 		(width 1)
 		(layer "F.Cu")
@@
 	)
 	(segment
-		(start 160.02 88.9)
-		(end 160.02 93.98)
+		(start 167.64 104.14)
+		(end 165.1 101.6)
 		(width 1)
 		(layer "F.Cu")
@@
 	)
 	(segment
-		(start 167.64 104.14)
-		(end 165.1 101.6)
+		(start 165.1 101.6)
+		(end 165.1 88.9)
 		(width 1)
 		(layer "F.Cu")
@@
 	)
 	(segment
-		(start 132.08 93.98)
-		(end 132.08 86.36)
+		(start 124.46 109.22)
+		(end 124.46 114.84)
 		(width 1)
 		(layer "F.Cu")
@@
 	)
 	(segment
-		(start 165.1 101.6)
-		(end 165.1 88.9)
+		(start 119.38 111.76)
+		(end 119.38 96.52)
 		(width 1)
 		(layer "F.Cu")
@@
 	)
 	(segment
-		(start 124.46 109.22)
-		(end 124.46 114.84)
+		(start 152.4 88.9)
+		(end 144.78 81.28)
 		(width 1)
 		(layer "F.Cu")
@@
 	)
 	(segment
-		(start 144.78 81.28)
-		(end 124.46 81.28)
+		(start 124.46 116.84)
+		(end 119.38 111.76)
 		(width 1)
 		(layer "F.Cu")
@@
 	)
 	(segment
-		(start 121.92 83.82)
-		(end 121.92 93.98)
+		(start 170.18 93.98)
+		(end 170.18 83.82)
 		(width 1)
 		(layer "F.Cu")
@@
 	)
 	(segment
-		(start 170.18 93.98)
-		(end 170.18 83.82)
+		(start 177.8 93.98)
+		(end 177.8 90.17)
 		(width 1)
 		(layer "F.Cu")
@@
 	)
 	(segment
-		(start 177.8 93.98)
-		(end 177.8 90.17)
+		(start 121.92 83.82)
+		(end 121.92 86.36)
 		(width 1)
 		(layer "F.Cu")
@@
 	)
 	(segment
-		(start 124.46 116.84)
-		(end 119.38 111.76)
-		(width 1)
-		(layer "F.Cu")
-		(net 0)
-	)
-	(segment
 		(start 165.1 88.9)
 		(end 167.64 86.36)
@@
 	)
 	(segment
-		(start 132.08 86.36)
-		(end 134.62 83.82)
+		(start 172.72 91.44)
+		(end 172.72 83.82)
 		(width 1)
 		(layer "F.Cu")
@@
 	)
 	(segment
-		(start 129.54 96.52)
-		(end 132.08 93.98)
+		(start 177.8 97.79)
+		(end 176.53 96.52)
 		(width 1)
 		(layer "F.Cu")
@@
 	)
 	(segment
-		(start 152.4 88.9)
-		(end 144.78 81.28)
+		(start 167.64 86.36)
+		(end 167.64 83.82)
 		(width 1)
 		(layer "F.Cu")
@@
 	)
 	(segment
-		(start 172.72 91.44)
-		(end 172.72 83.82)
+		(start 129.54 88.9)
+		(end 134.62 83.82)
 		(width 1)
 		(layer "F.Cu")
@@
 	)
 	(segment
-		(start 177.8 97.79)
-		(end 176.53 96.52)
+		(start 144.78 81.28)
+		(end 124.46 81.28)
 		(width 1)
 		(layer "F.Cu")
@@
 	)
 	(segment
-		(start 119.38 111.76)
-		(end 119.38 104.14)
+		(start 157.48 96.52)
+		(end 157.48 104.14)
 		(width 1)
 		(layer "F.Cu")
@@
 	)
 	(segment
-		(start 167.64 86.36)
-		(end 167.64 83.82)
-		(width 1)
-		(layer "F.Cu")
-		(net 0)
-	)
-	(segment
-		(start 157.48 96.52)
-		(end 157.48 104.14)
+		(start 134.62 83.82)
+		(end 137.16 83.82)
 		(width 1)
 		(layer "F.Cu")
@@
 	)
 	(segment
-		(start 144.78 81.28)
-		(end 129.54 81.28)
+		(start 152.4 86.36)
+		(end 149.86 88.9)
 		(width 1)
 		(layer "B.Cu")
@@
 	(segment
 		(start 132.08 109.22)
-		(end 132.08 104.14)
+		(end 132.08 96.52)
 		(width 1)
 		(layer "B.Cu")
@@
 	)
 	(segment
-		(start 172.72 99.06)
-		(end 170.18 101.6)
+		(start 137.16 121.92)
+		(end 134.62 119.38)
 		(width 1)
 		(layer "B.Cu")
@@
 	)
 	(segment
-		(start 147.32 83.82)
-		(end 144.78 81.28)
+		(start 134.62 119.38)
+		(end 134.62 111.76)
 		(width 1)
 		(layer "B.Cu")
@@
 	)
 	(segment
-		(start 172.72 88.9)
-		(end 172.72 99.06)
+		(start 172.72 99.06)
+		(end 170.18 101.6)
 		(width 1)
 		(layer "B.Cu")
@@
 	)
 	(segment
-		(start 134.62 109.22)
-		(end 134.62 96.52)
+		(start 147.32 83.82)
+		(end 144.78 81.28)
 		(width 1)
 		(layer "B.Cu")
@@
 	)
 	(segment
-		(start 170.18 101.6)
-		(end 167.64 101.6)
+		(start 127 83.82)
+		(end 127 88.9)
 		(width 1)
 		(layer "B.Cu")
@@
 	)
 	(segment
-		(start 132.08 104.14)
-		(end 129.54 101.6)
+		(start 149.86 88.9)
+		(end 149.86 119.38)
 		(width 1)
 		(layer "B.Cu")
@@
 	)
 	(segment
-		(start 134.62 111.76)
-		(end 132.08 109.22)
+		(start 172.72 88.9)
+		(end 172.72 99.06)
 		(width 1)
 		(layer "B.Cu")
@@
 	)
 	(segment
-		(start 134.62 96.52)
-		(end 132.08 93.98)
+		(start 132.08 86.36)
+		(end 129.54 86.36)
 		(width 1)
 		(layer "B.Cu")
@@
 	)
 	(segment
-		(start 147.32 121.92)
-		(end 137.16 121.92)
+		(start 134.62 88.9)
+		(end 132.08 86.36)
 		(width 1)
 		(layer "B.Cu")
@@
 	)
 	(segment
-		(start 134.62 119.38)
-		(end 134.62 111.76)
+		(start 170.18 101.6)
+		(end 167.64 101.6)
 		(width 1)
 		(layer "B.Cu")
@@
 	)
 	(segment
-		(start 149.86 119.38)
-		(end 147.32 121.92)
-		(width 1)
-		(layer "B.Cu")
-		(net 0)
-	)
-	(segment
 		(start 129.54 81.28)
 		(end 127 83.82)
@@
 	)
 	(segment
-		(start 152.4 86.36)
-		(end 149.86 88.9)
+		(start 132.08 96.52)
+		(end 129.54 93.98)
 		(width 1)
 		(layer "B.Cu")
@@
 	)
 	(segment
-		(start 132.08 93.98)
-		(end 129.54 93.98)
+		(start 134.62 111.76)
+		(end 132.08 109.22)
 		(width 1)
 		(layer "B.Cu")
@@
 	)
 	(segment
-		(start 127 96.52)
-		(end 129.54 99.06)
+		(start 127 88.9)
+		(end 129.54 91.44)
 		(width 1)
 		(layer "B.Cu")
@@
 	)
 	(segment
-		(start 127 83.82)
-		(end 127 96.52)
+		(start 144.78 81.28)
+		(end 129.54 81.28)
 		(width 1)
 		(layer "B.Cu")
@@
 	)
 	(segment
-		(start 149.86 88.9)
-		(end 149.86 119.38)
+		(start 152.4 83.82)
+		(end 147.32 83.82)
 		(width 1)
 		(layer "B.Cu")
@@
 	)
 	(segment
-		(start 152.4 83.82)
-		(end 147.32 83.82)
+		(start 147.32 121.92)
+		(end 137.16 121.92)
+		(width 1)
+		(layer "B.Cu")
+		(net 0)
+	)
+	(segment
+		(start 149.86 119.38)
+		(end 147.32 121.92)
 		(width 1)
 		(layer "B.Cu")
@@
 	)
 	(segment
-		(start 137.16 121.92)
-		(end 134.62 119.38)
+		(start 134.62 109.22)
+		(end 134.62 88.9)
 		(width 1)
 		(layer "B.Cu")

Commit message: adjust position of test LED
Parts:
- moved REF** 5.08 mm to (182.9, 87.6)
Routing:
- net (no net): track 413.8 -> 419.5 mm
Changed lines of the file:
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@@
 	(footprint "LED_THT:LED_D5.0mm"
 		(layer "F.Cu")
-		(at 177.8 87.63 -90)
+		(at 182.88 87.63 -90)
 		(descr "LED, diameter 5.0mm, 2 pins, http://cdn-reichelt.de/documents/datenblatt/A500/LL-504BC2E-009.pdf")
 		(tags "LED diameter 5.0mm 2 pins")
@@
 	)
 	(gr_text "Test LED"
-		(at 179.07 92.71 0)
+		(at 182.88 92.71 0)
 		(layer "F.SilkS")
 		(effects
@@
 				(thickness 0.1)
 			)
-			(justify left)
 		)
 	)
@@
 	)
 	(segment
+		(start 181.61 87.63)
+		(end 182.88 87.63)
+		(width 1)
+		(layer "F.Cu")
+		(net 0)
+	)
+	(segment
 		(start 175.26 93.98)
 		(end 172.72 91.44)
@@
 	)
 	(segment
+		(start 177.8 93.98)
+		(end 181.61 90.17)
+		(width 1)
+		(layer "F.Cu")
+		(net 0)
+	)
+	(segment
 		(start 160.02 88.9)
 		(end 160.02 93.98)
@@
 	)
 	(segment
+		(start 181.61 90.17)
+		(end 182.88 90.17)
+		(width 1)
+		(layer "F.Cu")
+		(net 0)
+	)
+	(segment
 		(start 119.38 111.76)
 		(end 119.38 96.52)
@@
 	)
 	(segment
-		(start 177.8 83.82)
-		(end 177.8 87.63)
-		(width 1)
-		(layer "F.Cu")
-		(net 0)
-	)
-	(segment
 		(start 170.18 93.98)
 		(end 170.18 83.82)
@@
 	)
 	(segment
-		(start 177.8 93.98)
-		(end 177.8 90.17)
-		(width 1)
-		(layer "F.Cu")
-		(net 0)
-	)
-	(segment
 		(start 121.92 83.82)
 		(end 121.92 86.36)
@@
 		(width 1)
 		(layer "F.Cu")
+		(net 0)
+	)
+	(segment
+		(start 177.8 83.82)
+		(end 181.61 87.63)
+		(width 1)
+		(layer "F.Cu")
